File: hardware/keys-group.kicad_sch (KiCad schematic)
At the start: 16 parts

Commit message: :construction: explode saki
Parts:
- added SW1: ~, KeysDock:KD-SINGLE-KEY, symbol components:KD_SINGLE_KEY
- renumbered SW1 to SW16
Connections:
- net LED_DATA_INNER: now also SW1.L2 (LED_DI); no longer SW16.L2 (LED_IN)
- net P,+3.3: now also SW1.H1 (HE_V3.3)
- net P,+5: now also SW1.L3 (LED_V5)
- net SAKI_MOVE: now also SW1.H6 (HE_AWAKE)
- net at SW13.H5 (GND), SW13.L1 (GND), SW14.H2 (GND)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: now also SW1.H2 (GND), SW1.H5 (GND), SW1.L1 (GND)
- net at T1.23 (Y8): now also SW1.H3 (HE_VOUT); no longer SW16.H3 (HE_VOUT)
- net at SW16.L2 (LED_DI): now also SW1.L4 (LED_DO); no longer SW16.L4 (LED_OUT)
- net LED_DATA_IN renamed TOMO0_IN
- net LED_DATA_OUT renamed TOMO0_OUT
- net SLEEP renamed RANA
- net RANA: now also SW1.H4 (HE_SLEEP)
Changed lines of the file:
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@@
 	(wire
 		(pts
-			(xy 186.69 96.52) (xy 186.69 104.14)
+			(xy 181.61 96.52) (xy 181.61 109.22)
 		)
 		(stroke
@@
 	(wire
 		(pts
-			(xy 200.66 96.52) (xy 186.69 96.52)
+			(xy 200.66 96.52) (xy 181.61 96.52)
 		)
 		(stroke
@@
 		)
 	)
-	(global_label "SLEEP"
+	(global_label "RANA"
 		(shape input)
 		(at 393.7 73.66 0)
@@
 		)
 		(property "Intersheetrefs" "${INTERSHEET_REFS}"
-			(at 402.4908 73.66 0)
+			(at 401.4629 73.66 0)
 			(effects
 				(font
@@
 		)
 	)
-	(global_label "SLEEP"
+	(global_label "RANA"
 		(shape input)
 		(at 393.7 152.4 0)
@@
 		)
 		(property "Intersheetrefs" "${INTERSHEET_REFS}"
-			(at 402.4908 152.4 0)
+			(at 401.4629 152.4 0)
 			(effects
 				(font
@@
 		)
 	)
-	(hierarchical_label "LED_DATA_OUT"
+	(hierarchical_label "TOMO0_OUT"
 		(shape output)
 		(at 34.29 168.91 180)
@@
 		)
 	)
-	(hierarchical_label "LED_DATA_IN"
+	(hierarchical_label "TOMO0_IN"
 		(shape input)
 		(at 387.35 54.61 0)
@@
 	(symbol
 		(lib_id "PCM_Generic:P,E")
-		(at 186.69 104.14 0)
+		(at 181.61 109.22 0)
 		(unit 1)
 		(exclude_from_sim no)
@@
 		(fields_autoplaced yes)
 		(property "Reference" "#PWR026"
-			(at 190.5 100.33 0)
+			(at 185.42 105.41 0)
 			(effects
 				(font
@@
 		)
 		(property "Value" "P,E"
-			(at 190.5 104.14 0)
+			(at 185.42 109.22 0)
 			(effects
 				(font
@@
 		)
 		(property "Footprint" ""
-			(at 186.69 104.14 0)
+			(at 181.61 109.22 0)
 			(effects
 				(font
@@
 		)
 		(property "Datasheet" ""
-			(at 186.69 104.14 0)
+			(at 181.61 109.22 0)
 			(effects
 				(font
@@
 		)
 		(property "Description" "earth/ground/earthing/grounding (E)"
-			(at 186.69 104.14 0)
+			(at 181.61 109.22 0)
 			(effects
 				(font
@@
 		(dnp no)
 		(fields_autoplaced yes)
-		(property "Reference" "#PWR"
+		(property "Reference" "#PWR0103"
 			(at 38.1 77.47 0)
 			(effects
@@
 					(unit 1)
 				)
+				(path "/6f5c986f-c08b-45be-b317-11f83a8063e7/abc5fe71-c02d-4ebe-9340-52eb4644c520"
+					(reference "#PWR0103")
+					(unit 1)
+				)
 			)
 		)
@@
 		(dnp no)
 		(fields_autoplaced yes)
-		(property "Reference" "#PWR"
+		(property "Reference" "#PWR0101"
 			(at 374.65 34.29 0)
 			(effects
@@
 					(unit 1)
 				)
+				(path "/6f5c986f-c08b-45be-b317-11f83a8063e7/abc5fe71-c02d-4ebe-9340-52eb4644c520"
+					(reference "#PWR0101")
+					(unit 1)
+				)
 			)
 		)
@@
 		(dnp no)
 		(fields_autoplaced yes)
-		(property "Reference" "#PWR"
+		(property "Reference" "#PWR0102"
 			(at 384.81 41.91 0)
 			(effects
@@
 					(unit 1)
 				)
+				(path "/6f5c986f-c08b-45be-b317-11f83a8063e7/abc5fe71-c02d-4ebe-9340-52eb4644c520"
+					(reference "#PWR0102")
+					(unit 1)
+				)

Commit message: :construction: sync components
Connections:
- net P,E: now also SW10.H2 (GND), SW10.H5 (GND), SW10.L1 (GND), SW11.H2 (GND), SW11.H5 (GND), SW11.L1 (GND), SW12.H2 (GND), SW12.H5 (GND), SW12.L1 (GND), SW2.H2 (GND), SW2.H5 (GND), SW2.L1 (GND), SW3.H2 (GND), SW3.H5 (GND), SW3.L1 (GND), SW4.H2 (GND), SW4.H5 (GND), SW4.L1 (GND), SW5.H2 (GND), SW5.H5 (GND), SW5.L1 (GND), SW9.H5 (GND), SW9.L1 (GND); no longer SW13.H2 (GND)
- now unconnected: SW1.H2 (GND), SW1.H5 (GND), SW1.L1 (GND), SW13.H5 (GND), SW13.L1 (GND), SW14.H2 (GND), SW14.H5 (GND), SW14.L1 (GND), SW15.H2 (GND), SW15.H5 (GND), SW15.L1 (GND), SW16.H2 (GND), SW16.H5 (GND), SW16.L1 (GND), SW6.H2 (GND), SW6.H5 (GND), SW6.L1 (GND), SW7.H2 (GND), SW7.H5 (GND), SW7.L1 (GND), SW8.H2 (GND), SW8.H5 (GND), SW8.L1 (GND)
Other:
- moved on the sheet: SW1, SW10, SW11, SW12, SW13, SW14, SW15, SW16, SW2, SW3, SW4, SW5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
