File: hardware/keys-group.kicad_sch (KiCad schematic)
At the start: 17 parts

Commit message: :art: improve LED positions
Parts:
- renumbered SW5 to SW?, SW7 to SW?, SW3 to SW?, SW4 to SW?, SW16 to SW?, SW1 to SW?, SW11 to SW?, SW10 to SW?, SW9 to SW?, SW2 to SW?, SW14 to SW?, SW12 to SW?, SW13 to SW?, SW6 to SW?, SW15 to SW?, SW8 to SW?, T1 to T?
Changed lines of the file:
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@@
 	(title_block
 		(title "Keys Dock Keys Group")
-		(date "2025-11-16")
-		(rev "0.2.6")
+		(date "2026-01-06")
+		(rev "0.2.7")
 		(company "keys.woooo.tech")
 	)
@@
 		(dnp no)
 		(fields_autoplaced yes)
-		(property "Reference" "#PWR026"
+		(property "Reference" "#PWR?"
 			(at 185.42 105.41 0)
 			(effects
@@
 		(dnp no)
 		(fields_autoplaced yes)
-		(property "Reference" "SW5"
+		(property "Reference" "SW?"
 			(at 359.41 40.64 0)
 			(effects
@@
 		(dnp no)
 		(fields_autoplaced yes)
-		(property "Reference" "SW7"
+		(property "Reference" "SW?"
 			(at 186.69 185.42 0)
 			(effects
@@
 		(dnp no)
 		(fields_autoplaced yes)
-		(property "Reference" "SW3"
+		(property "Reference" "SW?"
 			(at 186.69 40.64 0)
 			(effects
@@
 		(on_board yes)
 		(dnp no)
-		(property "Reference" "#PWR06"
+		(property "Reference" "#PWR?"
 			(at 386.08 134.62 0)
 			(effects
@@
 		(dnp no)
 		(fields_autoplaced yes)
-		(property "Reference" "SW4"
+		(property "Reference" "SW?"
 			(at 273.05 40.64 0)
 			(effects
@@
 		(dnp no)
 		(fields_autoplaced yes)
-		(property "Reference" "SW16"
+		(property "Reference" "SW?"
 			(at 316.23 185.42 0)
 			(effects
@@
 		(on_board yes)
 		(dnp no)
-		(property "Reference" "SW1"
+		(property "Reference" "SW?"
 			(at 359.41 185.42 0)
 			(effects
@@
 		(dnp no)
 		(fields_autoplaced yes)
-		(property "Reference" "SW11"
+		(property "Reference" "SW?"
 			(at 229.87 40.64 0)
 			(effects
@@
 		(dnp no)
 		(fields_autoplaced yes)
-		(property "Reference" "T1"
+		(property "Reference" "T?"
 			(at 236.22 113.0299 90)
 			(effects
@@
 		(dnp no)
 		(fields_autoplaced yes)
-		(property "Reference" "SW10"
+		(property "Reference" "SW?"
 			(at 143.51 40.64 0)
 			(effects
@@
 		(dnp no)
 		(fields_autoplaced yes)
-		(property "Reference" "#PWR022"
+		(property "Reference" "#PWR?"
 			(at 250.19 121.92 0)
 			(effects
@@
 		(dnp no)
 		(fields_autoplaced yes)
-		(property "Reference" "SW9"
+		(property "Reference" "SW?"
 			(at 57.15 40.64 0)
 			(effects
@@
 		(dnp no)
 		(fields_autoplaced yes)
-		(property "Reference" "SW2"
+		(property "Reference" "SW?"
 			(at 100.33 40.64 0)
 			(effects
@@
 		(on_board yes)
 		(dnp no)
-		(property "Reference" "#PWR01"
+		(property "Reference" "#PWR?"
 			(at 39.37 90.17 0)
 			(effects
@@
 		(dnp no)
 		(fields_autoplaced yes)
-		(property "Reference" "SW14"
+		(property "Reference" "SW?"
 			(at 143.51 185.42 0)
 			(effects
@@
 		(dnp no)
 		(fields_autoplaced yes)
-		(property "Reference" "SW12"
+		(property "Reference" "SW?"
 			(at 316.23 40.64 0)
 			(effects
@@
 		(dnp no)
 		(fields_autoplaced yes)
-		(property "Reference" "SW13"
+		(property "Reference" "SW?"
 			(at 57.15 185.42 0)
 			(effects
@@
 		(dnp no)
 		(fields_autoplaced yes)
-		(property "Reference" "SW6"
+		(property "Reference" "SW?"
 			(at 100.33 185.42 0)
 			(effects
@@
 		(dnp no)
 		(fields_autoplaced yes)
-		(property "Reference" "SW15"
+		(property "Reference" "SW?"
 			(at 229.87 185.42 0)
 			(effects
@@
 		(dnp no)
 		(fields_autoplaced yes)
-		(property "Reference" "SW8"
+		(property "Reference" "SW?"
 			(at 273.05 185.42 0)
 			(effects
@@
 		(dnp no)
 		(fields_autoplaced yes)
-		(property "Reference" "#PWR02"
+		(property "Reference" "#PWR?"
 			(at 35.56 161.29 0)
 			(effects
@@
 		(dnp no)
 		(fields_autoplaced yes)
-		(property "Reference" "#PWR0102"
+		(property "Reference" "#PWR?"
 			(at 383.54 38.1 0)
 			(effects

Commit message: :sparkles: add bom table
Parts:
- SW1, SW10, SW11, SW12, SW13, SW14, SW15, SW16, SW2, SW3, SW4, SW5, SW6, SW7, SW8, SW9: renamed from SW?; value ~ -> SC4823S6-TR; LCSC (none) -> C52021064; Manufacturer (none) -> Semiment(赛卓)
- T1: renamed from T?; value ~ -> XL4067TS; LCSC (none) -> C41427445; Manufacturer (none) -> XINLUDA
