File: hardware/controller.kicad_pcb (KiCad board)
At the start: 4 copper layers, 32 x 93.3 mm, 20 parts, among them J1 Connector, USB-TYPE-C-16P, U1 ESP32-C6-WROOM-1, U3 TPS62840YBGR

Commit message: 👆UPDATE SOME CONTROLLER LINE
Parts:
- moved R3 24.0 mm to (102.5, 117.5)
- moved C9 23.2 mm to (102.0, 115.0)
- moved L1 16.6 mm to (102.0, 108.0), turned to 180 degrees
- moved C8 14.9 mm to (99.0, 104.0)
- moved S2 11.4 mm to (96.0, 86.0), turned to -90 degrees
- moved U3 8.99 mm to (96.5, 109.0)
- moved C10 7.19 mm to (96.0, 102.5), turned to -90 degrees
- moved PC3 1.00 mm to (94.5, 135.0)
Routing:
- net /SAKI_MOVE: track 0.00 -> 91.3 mm
- net /KEYS_DT_3: track 0.00 -> 87.5 mm
- net /KEYS_DT_4: track 0.00 -> 87.0 mm
- net /KEYS_DT_1: track 0.00 -> 82.2 mm
- net /KEYS_DT_5: track 0.00 -> 78.9 mm
- net /KEYS_DT_2: track 0.00 -> 77.3 mm
- net /KEYS_CH_A: track 0.00 -> 62.8 mm, vias 0 -> 2
- net P,+3.3: track 8.30 -> 70.1 mm, vias 0 -> 2
- net /BOOT_1/RANA: track 0.00 -> 53.0 mm, vias 0 -> 1
- net /KEYS_CH_CE: track 0.00 -> 22.2 mm, vias 0 -> 1
- net /RANA: track 0.00 -> 20.1 mm, vias 0 -> 1
- net P,+5: track 0.00 -> 18.8 mm
- net P,E: track 10.1 -> 28.4 mm
- net /BOOT_0/KEYS_CH_CE: track 0.00 -> 8.88 mm, vias 0 -> 2
- net Net-(S2-A): track 0.00 -> 6.31 mm

Commit message: :construction: controller board
Parts:
- added R2: 4.7kΩ, KeysDock:R_0402, F.Cu at (94.8, 59.8)
- added R4: 4.7kΩ, KeysDock:R_0402, F.Cu at (87.2, 59.8)
- added R5: 100Ω, KeysDock:R_0402, F.Cu at (89.8, 136.5)
- added R6: 4.7kΩ, KeysDock:R_0402, F.Cu at (84.8, 133.0)
- added S1: Reset, 160gf, KeysDock:SW_TS-1088-AR02016, F.Cu at (87.2, 138.8)
- C10, C8, C9, L1, R3, U3: moved to B.Cu
- S2: value Tactile Button, 160gf -> Joint Download, 160gf
- moved R1 50.9 mm to (91.2, 131.8), turned to 180 degrees
- moved S2 44.8 mm to (95.4, 130.8), turned to 0 degrees
- moved D1 38.0 mm to (96.0, 118.7), turned to -90 degrees
- moved D2 35.4 mm to (98.5, 118.7), turned to -90 degrees
- moved PC3 25.8 mm to (100.2, 109.9), turned to 180 degrees
- moved C9 24.9 mm to (98.1, 90.4)
- moved R3 23.6 mm to (94.8, 95.2), turned to 90 degrees
- moved L1 17.6 mm to (95.1, 91.8), turned to 90 degrees
- moved U3 16.2 mm to (97.8, 92.9), turned to 180 degrees
- moved C10 13.6 mm to (98.4, 89.2), turned to 0 degrees
- moved C8 8.70 mm to (96.2, 95.8), turned to 180 degrees
- moved C7 7.25 mm to (78.8, 131.2), turned to 0 degrees
- moved C6 3.66 mm to (78.8, 133.0), turned to 0 degrees
- moved C4 3.56 mm to (78.8, 136.5), turned to 0 degrees
- moved C5 0.25 mm to (78.8, 134.8), turned to 0 degrees
Connections:
- C10 pad 1: +3.3V -> P,+3.3
- C10 pad 2: GND -> P,E
- C8 pad 1: +5V -> P,+5
- C8 pad 2: GND -> P,E
- C9 pad 1: +3.3V -> P,+3.3
- C9 pad 2: GND -> P,E
- J1 pad A5: unconnected-(J1-CC1-PadA5) -> Net-(J1-CC1)
- J1 pad A6: unconnected-(J1-D+-PadA6) -> /USB_D+
- J1 pad A7: unconnected-(J1-D--PadA7) -> /USB_D-
- J1 pad A9B4: Net-(J1-VBUS-PadA9B4) -> P,+5
- J1 pad B5: unconnected-(J1-CC2-PadB5) -> Net-(J1-CC2)
- J1 pad B6: unconnected-(J1-D+-PadB6) -> /USB_D+
- J1 pad B7: unconnected-(J1-D--PadB7) -> /USB_D-
- J1 pad B9A4: Net-(J1-VBUS-PadA9B4) -> P,+5
- L1 pad 2: +3.3V -> P,+3.3
- R3 pad 1: GND -> P,E
- U3 pad A1: GND -> P,E
- U3 pad A2: +3.3V -> P,+3.3
- U3 pad B1: +5V -> P,+5
- U3 pad C1: +5V -> P,+5
Routing:
- net P,+5: track 18.8 -> 106.3 mm, vias 0 -> 5
- net /KEYS_CH_C: track 0.00 -> 82.0 mm, vias 0 -> 4
- net /USB_D+: track 0.00 -> 79.4 mm, vias 0 -> 2
- net /USB_D-: track 0.00 -> 77.5 mm, vias 0 -> 2
- net /KEYS_CH_D: track 0.00 -> 76.4 mm, vias 0 -> 4
- net /SWITCH: track 0.00 -> 75.4 mm, vias 0 -> 1
- net /KEYS_CH_B: track 0.00 -> 69.8 mm, vias 0 -> 4
- net /TOMO0: track 0.00 -> 69.1 mm, vias 0 -> 2
- net /WHEEL: track 0.00 -> 48.5 mm, vias 0 -> 2
- net /EINK_DC: track 0.00 -> 32.4 mm, vias 0 -> 1
- net /RANA: track 20.1 -> 51.4 mm
- net /BOOT_1/RANA: track 53.0 -> 22.0 mm
- net /EINK_SPI_MOSI: track 0.00 -> 29.0 mm, vias 0 -> 1
- net /KEYS_CH_CE: track 22.2 -> 51.0 mm, vias 1 -> 3
- net /U0TX: track 3.43 -> 31.3 mm
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- added copper zone on B.Cu, net P,E
- added copper zone on F.Cu, net P,E
- added copper zone on In1.Cu, net P,E
- added copper zone on In2.Cu, net P,E
Other:
- board text added: "(c) 2025 Wo0t3c Industries"
- board text added: "+ -"
- board text added: "5V 3.3V"
- board text added: "Designed by Reverier-Xu"
- board text added: "Ijichi Nijika"
- board text added: "KD-0.2.6-G7370F30-K9-RS91"
- board text added: "Keys Dock - Creating Reality with Idealism. -"
- board text added: "MODE"
- board text added: "RESET"
- board text added: "Switch & LED"
- board text added: "TX RX"
- board text added: "Type-C Out"
- board text added: "UART"
- board text added: "https://github.com/Reverier-Xu/KeysDock"
