File: hardware/typeboard.kicad_pcb (KiCad board)
At the start: 4 copper layers, 288.8 x 97.2 mm, 136 parts, among them J2 AXK6F20347YG

Commit message: :sparkles: finish all hardware designs except external
Other:
- board text added: "Controller"
- board text added: "Designed by Reverier-Xu, (c) 2026 Wo0t3c Industries"
- board text removed: "Designed by Reverier-Xu, (c) 2025 Wo0t3c Industries"
