File: hardware/external.kicad_pcb (KiCad board)
At the start: 2 copper layers, 285.8 x 21 mm, 20 parts

Commit message: :sparkles: finish pcb layout of controller
Parts:
- added R5: 100Ω, KeysDock:R_0402, B.Cu at (180.5, 100.5)
- moved SW12 200.0 mm to (90.5, 97.5)
- moved SW10 185.7 mm to (66.7, 97.5)
- moved SW1 161.9 mm to (228.6, 97.5)
- moved SW13 119.1 mm to (190.5, 97.5)
- moved SW5 104.8 mm to (252.4, 97.5)
- moved SW3 100.0 mm to (209.5, 97.5)
- moved SW2 81.0 mm to (171.4, 97.5)
- moved SW7 81.0 mm to (271.4, 97.5)
- moved SW8 81.0 mm to (128.6, 97.5)
- moved SW6 61.9 mm to (109.5, 97.5)
- moved SW9 61.9 mm to (290.5, 97.5)
- moved R3 60.0 mm to (219.0, 101.5)
- moved R4 47.4 mm to (206.4, 104.2), turned to -90 degrees
- moved T1 40.7 mm to (200.0, 92.5)
- moved SW11 38.1 mm to (309.5, 97.5)
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Connections:
- SW1 pad H2: P,E -> P,GND
- SW1 pad H4: unconnected-(SW1-HE_SLEEP-PadH4) -> Net-(SW1-HE_SLEEP)
- SW1 pad H5: P,E -> P,GND
- SW10 pad H2: P,E -> P,GND
- SW10 pad H5: P,E -> P,GND
- SW11 pad H2: P,E -> P,GND
- SW11 pad H4: unconnected-(SW1-HE_SLEEP-PadH4) -> Net-(SW1-HE_SLEEP)
- SW11 pad H5: P,E -> P,GND
- SW12 pad H2: P,E -> P,GND
- SW12 pad H5: P,E -> P,GND
- SW13 pad H2: P,E -> P,GND
- SW13 pad H4: unconnected-(SW1-HE_SLEEP-PadH4) -> Net-(SW1-HE_SLEEP)
- SW13 pad H5: P,E -> P,GND
- SW14 pad H2: P,E -> P,GND
- SW14 pad H4: unconnected-(SW1-HE_SLEEP-PadH4) -> Net-(SW1-HE_SLEEP)
- SW14 pad H5: P,E -> P,GND
- SW2 pad H2: P,E -> P,GND
- SW2 pad H5: P,E -> P,GND
- SW3 pad H2: P,E -> P,GND
- SW3 pad H4: unconnected-(SW1-HE_SLEEP-PadH4) -> Net-(SW1-HE_SLEEP)
- SW3 pad H5: P,E -> P,GND
- SW4 pad H2: P,E -> P,GND
- SW4 pad H5: P,E -> P,GND
- SW5 pad H2: P,E -> P,GND
- SW5 pad H4: unconnected-(SW1-HE_SLEEP-PadH4) -> Net-(SW1-HE_SLEEP)
- SW5 pad H5: P,E -> P,GND
- SW6 pad H2: P,E -> P,GND
- SW6 pad H5: P,E -> P,GND
- SW7 pad H2: P,E -> P,GND
- SW7 pad H4: unconnected-(SW1-HE_SLEEP-PadH4) -> Net-(SW1-HE_SLEEP)
- SW7 pad H5: P,E -> P,GND
- SW8 pad H2: P,E -> P,GND
- SW8 pad H5: P,E -> P,GND
- SW9 pad H2: P,E -> P,GND
- SW9 pad H4: unconnected-(SW1-HE_SLEEP-PadH4) -> Net-(SW1-HE_SLEEP)
- SW9 pad H5: P,E -> P,GND
- T1 pad 12: P,E -> P,GND
Routing:
- net P,+3.3: track 0.00 -> 328.7 mm, vias 0 -> 16
- net Net-(SW10-HE_VOUT): track 0.00 -> 137.9 mm
- net Net-(SW14-HE_VOUT): track 0.00 -> 135.0 mm
- net Net-(SW12-HE_VOUT): track 0.00 -> 115.8 mm
- net Net-(SW11-HE_VOUT): track 0.00 -> 112.7 mm
- net Net-(SW6-HE_VOUT): track 0.00 -> 94.6 mm
- net Net-(SW9-HE_VOUT): track 0.00 -> 91.3 mm
- net Net-(SW8-HE_VOUT): track 0.00 -> 75.3 mm
- net Net-(SW7-HE_VOUT): track 0.00 -> 72.0 mm
- net Net-(SW4-HE_VOUT): track 0.00 -> 56.0 mm
- net Net-(SW5-HE_VOUT): track 0.00 -> 52.7 mm
- net Net-(SW2-HE_VOUT): track 0.00 -> 31.6 mm
- net Net-(SW1-HE_VOUT): track 0.00 -> 28.6 mm
- net Net-(SW13-HE_VOUT): track 0.00 -> 28.5 mm, vias 0 -> 2
- net KEYS_ADC_OUT: track 0.00 -> 21.0 mm, vias 0 -> 2
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Other:
- outline, holes or cut-outs redrawn
- copper layers 2 -> 4

Commit message: :fire: remove CH-series chips and use legacy UART
Routing:
- net P,GND: track 0.00 -> 4.96 mm, vias 29 -> 30
- added copper zone on B.Cu, net P,E
- added copper zone on F.Cu, net P,E
- added copper zone on In1.Cu, net P,E
- added copper zone on In2.Cu, net P,GND
Changed lines of the file:
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@@
+	)
+	(via
+		(at 204.5 100.25)
+		(size 0.6)
+		(drill 0.3)
+		(layers "F.Cu" "B.Cu")
+		(net 12)
 	)
 	(via
@@
 		(drill 0.3)
 		(layers "F.Cu" "B.Cu")
+		(net 12)
+	)
+	(segment
+		(start 203 96.075)
+		(end 202.8 96.275)
+		(width 0.3)
+		(layer "B.Cu")
+		(net 12)
+	)
+	(segment
+		(start 202.8 98.55)
+		(end 204.5 100.25)
+		(width 0.3)
+		(layer "B.Cu")
+		(net 12)
+	)
+	(segment
+		(start 202.8 96.275)
+		(end 202.8 98.55)
+		(width 0.3)
+		(layer "B.Cu")
 		(net 12)
 	)
@@
 		(net 28)
 	)
+	(zone
+		(net 8)
+		(net_name "P,E")
+		(layers "F.Cu" "B.Cu" "In1.Cu")
+		(hatch edge 0.5)
+		(connect_pads yes
+			(clearance 0.5)
+		)
+		(min_thickness 0.25)
+		(filled_areas_thickness no)
+		(fill yes
+			(thermal_gap 0.5)
+			(thermal_bridge_width 0.5)
+		)
+		(polygon
+			(pts
+				(xy 56.75 87.5) (xy 343.25 87.5) (xy 343.25 107.5) (xy 56.75 107.5)
+			)
+		)
+	)
+	(zone
+		(net 12)
+		(net_name "P,GND")
+		(layer "In2.Cu")
+		(hatch edge 0.5)
+		(connect_pads yes
+			(clearance 0.5)
+		)
+		(min_thickness 0.25)
+		(filled_areas_thickness no)
+		(fill yes
+			(thermal_gap 0.5)
+			(thermal_bridge_width 0.5)
+		)
+		(polygon
+			(pts
+				(xy 56.75 87.5) (xy 343.25 87.5) (xy 343.25 107.5) (xy 56.75 107.5)
+			)
+		)
+	)
 	(group ""

Commit message: :sparkles: finish all hardware designs
Parts:
- moved R4 8.75 mm to (214.2, 108.0), turned to 0 degrees
- moved R5 2.55 mm to (181.0, 103.0)
- moved R3 1.50 mm to (219.0, 103.0)
Connections:
- SW10 pad H4: unconnected-(SW10-HE_SLEEP-PadH4) -> Net-(SW1-HE_SLEEP)
- SW12 pad H4: unconnected-(SW10-HE_SLEEP-PadH4) -> Net-(SW1-HE_SLEEP)
- SW2 pad H4: unconnected-(SW10-HE_SLEEP-PadH4) -> Net-(SW1-HE_SLEEP)
- SW4 pad H4: unconnected-(SW10-HE_SLEEP-PadH4) -> Net-(SW1-HE_SLEEP)
- SW6 pad H4: unconnected-(SW10-HE_SLEEP-PadH4) -> Net-(SW1-HE_SLEEP)
- SW8 pad H4: unconnected-(SW10-HE_SLEEP-PadH4) -> Net-(SW1-HE_SLEEP)
Routing:
- net Net-(SW1-HE_SLEEP): track 0.00 -> 373.3 mm, vias 8 -> 15
- net Net-(SW1-HE_AWAKE): track 0.00 -> 370.2 mm, vias 14 -> 37
- net P,+3.3: track 328.7 -> 331.2 mm, vias 16 -> 17
- net P,E: track 2.28 -> 0.00 mm, vias 2 -> 28
- net KEYS_CH_A: track 15.6 -> 16.9 mm
- net KEYS_CH_CE: track 16.6 -> 17.1 mm
- net unconnected-(SW10-HE_SLEEP-PadH4): vias 6 -> 0

Commit message: :sparkles: add silk tips for external board
Other:
- board text added: "DEL"
- board text added: "ESC"
- board text added: "F1"
- board text added: "F10"
- board text added: "F11"
- board text added: "F12"
- board text added: "F2"
- board text added: "F3"
- board text added: "F4"
- board text added: "F5"
- board text added: "F6"
- board text added: "F7"
- board text added: "F8"
- board text added: "F9"
Changed lines of the file:
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@@
 		(layer "User.1")
+	)
+	(gr_text "F5"
+		(at 166 92.75 0)
+		(layer "F.SilkS")
+		(effects
+			(font
+				(size 0.5 0.5)
+				(thickness 0.1)
+			)
+			(justify left bottom)
+		)
+	)
+	(gr_text "F1"
+		(at 85 92.75 0)
+		(layer "F.SilkS")
+		(effects
+			(font
+				(size 0.5 0.5)
+				(thickness 0.1)
+			)
+			(justify left bottom)
+		)
+	)
+	(gr_text "F4"
+		(at 142.25 92.75 0)
+		(layer "F.SilkS")
+		(effects
+			(font
+				(size 0.5 0.5)
+				(thickness 0.1)
+			)
+			(justify left bottom)
+		)
+	)
+	(gr_text "ESC"
+		(at 61.25 92.75 0)
+		(layer "F.SilkS")
+		(effects
+			(font
+				(size 0.5 0.5)
+				(thickness 0.1)
+			)
+			(justify left bottom)
+		)
+	)
+	(gr_text "F12"
+		(at 304 92.75 0)
+		(layer "F.SilkS")
+		(effects
+			(font
+				(size 0.5 0.5)
+				(thickness 0.1)
+			)
+			(justify left bottom)
+		)
+	)
+	(gr_text "F7"
+		(at 204 92.75 0)
+		(layer "F.SilkS")
+		(effects
+			(font
+				(size 0.5 0.5)
+				(thickness 0.1)
+			)
+			(justify left bottom)
+		)
+	)
+	(gr_text "F9"
+		(at 247 92.75 0)
+		(layer "F.SilkS")
+		(effects
+			(font
+				(size 0.5 0.5)
+				(thickness 0.1)
+			)
+			(justify left bottom)
+		)
+	)
+	(gr_text "DEL"
+		(at 328 92.75 0)
+		(layer "F.SilkS")
+		(effects
+			(font
+				(size 0.5 0.5)
+				(thickness 0.1)
+			)
+			(justify left bottom)
+		)
+	)
+	(gr_text "F11"
+		(at 285 92.75 0)
+		(layer "F.SilkS")
+		(effects
+			(font
+				(size 0.5 0.5)
+				(thickness 0.1)
+			)
+			(justify left bottom)
+		)
+	)
+	(gr_text "F2"
+		(at 104.25 92.75 0)
+		(layer "F.SilkS")
+		(effects
+			(font
+				(size 0.5 0.5)
+				(thickness 0.1)
+			)
+			(justify left bottom)
+		)
+	)
+	(gr_text "F6"
+		(at 185 92.75 0)
+		(layer "F.SilkS")
+		(effects
+			(font
+				(size 0.5 0.5)
+				(thickness 0.1)
+			)
+			(justify left bottom)
+		)
+	)
+	(gr_text "F10"
+		(at 266 92.75 0)
+		(layer "F.SilkS")
+		(effects
+			(font
+				(size 0.5 0.5)
+				(thickness 0.1)
+			)
+			(justify left bottom)
+		)
+	)
+	(gr_text "F8"
+		(at 223.25 92.75 0)
+		(layer "F.SilkS")
+		(effects
+			(font
+				(size 0.5 0.5)
+				(thickness 0.1)
+			)
+			(justify left bottom)
+		)
+	)
+	(gr_text "F3"
+		(at 123.25 92.75 0)
+		(layer "F.SilkS")
+		(effects
+			(font
+				(size 0.5 0.5)
+				(thickness 0.1)
+			)
+			(justify left bottom)
+		)
 	)
 	(segment
