File: hardware/external.kicad_pcb (KiCad board)
At the start: 4 copper layers, 285.8 x 21 mm, 21 parts

Commit message: :sparkles: add testboard
Parts:
- moved SW10 23.8 mm to (90.5, 97.5)
- moved SW12 23.8 mm to (66.7, 97.5)
- moved SW1 19.1 mm to (209.5, 97.5)
- moved SW3 19.1 mm to (228.6, 97.5)
- moved SW6 19.0 mm to (128.6, 97.5)
- moved SW8 19.0 mm to (109.5, 97.5)
Routing:
- net Net-(SW12-HE_VOUT): track 115.8 -> 137.9 mm
- net Net-(SW10-HE_VOUT): track 137.9 -> 115.8 mm
- net Net-(SW8-HE_VOUT): track 75.3 -> 94.6 mm
- net Net-(SW6-HE_VOUT): track 94.6 -> 75.3 mm
- net Net-(SW3-HE_VOUT): track 12.9 -> 28.6 mm
- net Net-(SW1-HE_VOUT): track 28.6 -> 12.9 mm
