File: hardware/external.kicad_pcb (KiCad board)
At the start: 4 copper layers, 285.8 x 21 mm, 21 parts

Commit message: :sparkles: add bom table
Parts:
- SW1, SW10, SW11, SW12, SW13, SW14, SW2, SW3, SW4, SW5, SW6, SW7, SW8, SW9: value ~ -> SC4823S6-TR
- T1: value ~ -> XL4067TS

Commit message: :construction: panelize all boards
Connections:
- PC1 pad 1: P,+3.3 -> /KEYS_CH_D
- PC1 pad 2: P,E -> /KEYS_CH_C
- PC1 pad 3: KEYS_ADC_OUT -> /KEYS_CH_B
- PC1 pad 4: KEYS_CH_CE -> /KEYS_CH_A
- PC1 pad 5: KEYS_CH_A -> /KEYS_CH_CE
- PC1 pad 6: KEYS_CH_B -> /KEYS_ADC_OUT
- PC1 pad 7: KEYS_CH_C -> P,E
- PC1 pad 8: KEYS_CH_D -> P,+3.3
- T1 pad 1: KEYS_ADC_OUT -> /KEYS_ADC_OUT
- T1 pad 10: KEYS_CH_A -> /KEYS_CH_A
- T1 pad 11: KEYS_CH_B -> /KEYS_CH_B
- T1 pad 13: KEYS_CH_D -> /KEYS_CH_D
- T1 pad 14: KEYS_CH_C -> /KEYS_CH_C
- T1 pad 15: KEYS_CH_CE -> /KEYS_CH_CE
Routing:
- net /KEYS_ADC_OUT: track 0.00 -> 23.3 mm, vias 0 -> 2
- net KEYS_ADC_OUT: track 21.0 -> 0.00 mm, vias 2 -> 0
- net /KEYS_CH_D: track 0.00 -> 20.5 mm, vias 0 -> 2
- net /KEYS_CH_C: track 0.00 -> 19.2 mm, vias 0 -> 2
- net KEYS_CH_CE: track 17.1 -> 0.00 mm, vias 2 -> 0
- net KEYS_CH_A: track 16.9 -> 0.00 mm, vias 2 -> 0
- net KEYS_CH_B: track 15.5 -> 0.00 mm
- net KEYS_CH_C: track 15.3 -> 0.00 mm
- net /KEYS_CH_CE: track 0.00 -> 14.8 mm
- net /KEYS_CH_A: track 0.00 -> 14.5 mm
- net /KEYS_CH_B: track 0.00 -> 13.7 mm
- net KEYS_CH_D: track 13.5 -> 0.00 mm
- net Net-(SW13-HE_VOUT): track 28.5 -> 27.4 mm
