File: hardware/testpad.kicad_pcb (KiCad board)
At the start: 2 copper layers, 11.8 x 8.8 mm, 13 parts, among them U2 ESP32-C6-WROOM-1, U3 TPS62840YBGR

Commit message: :art: improve LED positions
Parts:
- removed C1: 4.7uF, KeysDock:C_0402
- removed C2: 10uF, KeysDock:C_0402
- removed C3: 22uF, KeysDock:C_0603
- removed L1: 22uH,5mA, KeysDock:IND-SMD_L2.5-W2.0_MHCHL2520
- removed R1: 10kΩ, KeysDock:R_0402
- removed R3: 267kΩ, KeysDock:R_0402
- removed S1: Tactile Button, 160gf, KeysDock:SW_TS-1088-AR02016
- removed SW1, SW2, SW3, SW4: ~, KeysDock:KD-SINGLE-KEY
- removed U2: ESP32-C6-WROOM-1, PCM_Espressif:ESP32-C6-WROOM-1
- removed U3: TPS62840YBGR, KeysDock:BGA6N40P3X2_146X96X50N
Other:
- board outline removed

Commit message: :sparkles: add testboard
Parts:
- added C1: 4.7uF, KeysDock:C_0402, B.Cu at (75.0, 81.2)
- added C10: 22uF, KeysDock:C_0402, B.Cu at (87.5, 78.1)
- added C11: 1uF, KeysDock:C_0402, B.Cu at (81.8, 71.2)
- added C14: 4.7uF, KeysDock:C_0402, B.Cu at (81.0, 81.2)
- added C15: 1uF, KeysDock:C_0402, B.Cu at (80.0, 84.2)
- added C2: 1uF, KeysDock:C_0402, B.Cu at (82.8, 71.2)
- added C3: 1uF, KeysDock:C_0402, B.Cu at (83.3, 72.9)
- added C4: 100nF, KeysDock:C_0402, B.Cu at (69.8, 131.2)
- added C5: 100nF, KeysDock:C_0402, B.Cu at (69.8, 130.2)
- added C6: 100nF, KeysDock:C_0402, B.Cu at (69.8, 129.2)
- added C7: 100nF, KeysDock:C_0402, B.Cu at (69.8, 128.2)
- added C8: 10uF, KeysDock:C_0402, B.Cu at (82.5, 78.8)
- added C9: 3.3nF, KeysDock:C_0402, B.Cu at (84.1, 83.8)
- added D1: SM4007PL, KeysDock:D_SOD-123FL, B.Cu at (71.0, 62.6)
- added J1: Connector, USB-TYPE-C-16P, KeysDock:HC-TYPE-C-16P-CB1.6, B.Cu at (82.0, 47.2)
- added J3: AFA01-S08FCA-00, KeysDock:AFA01-S08FCA-00, F.Cu at (82.2, 95.2)
- added L1: 2.2uH,5mA, KeysDock:IND-SMD_L2.5-W2.0_MHCHL2520, B.Cu at (90.0, 79.2)
- added LED1: ~, KeysDock:XL-3512RGBW-WS2812B, F.Cu at (65.4, 67.1)
- added LED2: ~, KeysDock:XL-6028RGBW-WS2812B, F.Cu at (103.0, 128.8)
- added LED3: ~, KeysDock:XL-6028RGBW-WS2812B, F.Cu at (103.0, 109.7)
- added LED4: ~, KeysDock:XL-6028RGBW-WS2812B, F.Cu at (103.0, 90.7)
- added LED5: ~, KeysDock:XL-6028RGBW-WS2812B, F.Cu at (103.0, 71.6)
- added PC1: ~, KeysDock:HC-1.25-4PWT, B.Cu at (89.1, 107.0)
- added PC2: ~, KeysDock:HC-1.25-2PWT, B.Cu at (91.5, 89.7)
- added R1: 10kΩ, KeysDock:R_0402, B.Cu at (75.5, 83.7)
- added R10: 0Ω, KeysDock:R_0402, B.Cu at (65.8, 57.7)
- added R11: 3kΩ, KeysDock:R_0402, B.Cu at (78.0, 84.2)
- added R12: 10kΩ, KeysDock:R_0402, F.Cu at (76.8, 55.2)
- added R13: 100Ω, KeysDock:R_0402, F.Cu at (67.0, 69.2)
- added R14: 100Ω, KeysDock:R_0402, B.Cu at (101.5, 66.2)
- added R2: 4.7kΩ, KeysDock:R_0402, B.Cu at (86.2, 53.2)
- added R3: 100kΩ, KeysDock:R_0402, B.Cu at (87.4, 83.3)
- added R4: 4.7kΩ, KeysDock:R_0402, B.Cu at (77.8, 53.2)
- added R5: 100Ω, KeysDock:R_0402, B.Cu at (70.3, 69.8)
- added R6: 100Ω, KeysDock:R_0402, B.Cu at (88.5, 98.2)
- added R7: 1.78kΩ, KeysDock:R_0402, B.Cu at (77.0, 84.2)
- added R8: 1.54kΩ, KeysDock:R_0402, B.Cu at (81.5, 82.7)
- added R9: 10kΩ, KeysDock:R_0402, F.Cu at (87.2, 55.2)
- added S1: Reset, 160gf, KeysDock:TS24CA, B.Cu at (66.2, 71.5)
- added S2: ~, KeysDock:EC12E1240301, F.Cu at (82.0, 63.2)
- added S3: Joint Download, 160gf, KeysDock:SW_TS-1088-AR02016, B.Cu at (84.0, 97.7)
- added SW1: ~, KeysDock:SW-SMD_SSSS811101, B.Cu at (67.0, 63.5)
- added SW2: ~, KeysDock:KD-SINGLE-KEY, F.Cu at (107.5, 128.8)
- added SW3: ~, KeysDock:KD-SINGLE-KEY, F.Cu at (107.5, 109.7)
- added SW4: ~, KeysDock:KD-SINGLE-KEY, F.Cu at (107.5, 90.7)
- added SW5: ~, KeysDock:KD-SINGLE-KEY, F.Cu at (107.5, 71.6)
- added T1: ~, KeysDock:XL4067TS, B.Cu at (107.5, 58.0)
- added U1: ESP32-C6-WROOM-1, KeysDock:ESP32-C6-WROOM-1, B.Cu at (82.0, 125.7)
- added U2: BQ24074RGTR, KeysDock:QFN50P300X300X80-17N, B.Cu at (78.0, 80.7)
- added U3: TLA2518IRTER, KeysDock:QFN50P300X300X80-17N, B.Cu at (85.5, 70.2)
- added U6: TPS62142RGTR, KeysDock:QFN50P300X300X80-17N, B.Cu at (85.5, 80.7)
Routing:
- net P,+3.3: track 0.00 -> 303.1 mm, vias 0 -> 13
- net /SAKI_MOVE: track 0.00 -> 182.0 mm, vias 0 -> 14
- net /RANA: track 0.00 -> 181.4 mm, vias 0 -> 5
- net P,+5: track 0.00 -> 143.4 mm, vias 0 -> 12
- net /TOMO0: track 0.00 -> 117.7 mm, vias 0 -> 1
- net /KEYS_CH_B: track 0.00 -> 93.0 mm, vias 0 -> 4
- net /KEYS_CH_A: track 0.00 -> 91.0 mm, vias 0 -> 4
- net /USB_PWR_SUPP: track 0.00 -> 86.1 mm, vias 0 -> 8
- net /USB_D-: track 0.00 -> 85.0 mm, vias 0 -> 2
- net /WHEEL_A: track 0.00 -> 84.2 mm, vias 0 -> 7
- net /USB_D+: track 0.00 -> 84.0 mm, vias 0 -> 2
- net /WHEEL_B: track 0.00 -> 82.3 mm, vias 0 -> 7
- net /KEYS_CH_C: track 0.00 -> 81.1 mm, vias 0 -> 2
- net Net-(SW2-HE_VOUT): track 0.00 -> 79.1 mm
- net /KEYS_CH_CE: track 0.00 -> 78.8 mm, vias 0 -> 2
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- added copper zone on B.Cu, net P,E
- added copper zone on F.Cu, net P,E
- added copper zone on In1.Cu, net P,E
- added copper zone on In2.Cu, net P,GND
Other:
- board outline added: 54.5 x 93.2 mm
- copper layers 2 -> 4
- board text added: "(c) 2026 Wo0t3c Industries"
- board text added: "+ -"
- board text added: "-0 TX RX +5"
- board text added: "BAT"
- board text added: "Designed by Reverier-Xu"
- board text added: "E-INK"
- board text added: "ESP32-C6"
- board text added: "Ijichi Nijika"
- board text added: "Keys Dock"
- board text added: "RESET"
- board text added: "Switch & LED"
- board text added: "Typeboard"
- board text added: "[KEYS] [@]$ _"

Commit message: :sparkles: add bom table
Parts:
- J1: value Connector, USB-TYPE-C-16P -> HC-TYPE-C-16P-CB1.6
- LED1: value ~ -> XL-3512RGBW-WS2812B
- LED2, LED3, LED4, LED5: value ~ -> XL-6028RGBW-WS2812B
- PC1: value ~ -> HC-1.25-4PWT
- PC2: value ~ -> HC-1.25-2PWT
- S1: value Reset, 160gf -> TS24CA
- S2: value ~ -> EC12E1240301
- S3: value Joint Download, 160gf -> TS-1088-AR02016, 160gf
- SW1: value ~ -> SSSS811101
- SW2, SW3, SW4, SW5: value ~ -> SC4823S6-TR
- T1: value ~ -> XL4067TS
- U1: value ESP32-C6-WROOM-1 -> ESP32-C6-WROOM-1-N8
