File: hardware/connector.kicad_sch (KiCad schematic)
At the start: 2 parts, among them J1 AXK5F20347YG, J2 AXK5F20347YG

Commit message: :sparkles: assembly all the part!
Other:
- moved on the sheet: J1, J2

Commit message: :sparkles: add bom table
Parts:
- J1, J2: LCSC (none) -> C3644763; Manufacturer (none) -> Panasonic; PartNumber (none) -> AXK-5F20347YG
Changed lines of the file:
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@@
+			)
+		)
+		(property "Manufacturer" "Panasonic"
+			(at 125.73 592.71 0)
+			(effects
+				(font
+					(size 1.27 1.27)
+				)
+				(justify left top)
+				(hide yes)
+			)
+		)
+		(property "PartNumber" "AXK-5F20347YG"
+			(at 125.73 692.71 0)
+			(effects
+				(font
+					(size 1.27 1.27)
+				)
+				(justify left top)
+				(hide yes)
+			)
+		)
+		(property "LCSC" "C3644763"
+			(at 106.68 97.79 0)
+			(effects
+				(font
+					(size 1.27 1.27)
+				)
+				(hide yes)
 			)
 		)
@@
 				(hide yes)
 			)
+		)
+		(property "Manufacturer" "Panasonic"
+			(at 170.18 592.71 0)
+			(effects
+				(font
+					(size 1.27 1.27)
+				)
+				(justify left top)
+				(hide yes)
+			)
+		)
+		(property "PartNumber" "AXK-5F20347YG"
+			(at 170.18 692.71 0)
+			(effects
+				(font
+					(size 1.27 1.27)
+				)
+				(justify left top)
+				(hide yes)
+			)
+		)
+		(property "LCSC" "C3644763"
+			(at 189.23 97.79 0)
+			(effects
+				(font
+					(size 1.27 1.27)
+				)
+				(hide yes)
+			)
