File: hardware/external.kicad_sch (KiCad schematic)
At the start: 21 parts, among them SW1 SC4823S6-TR, SW10 SC4823S6-TR, SW11 SC4823S6-TR, SW12 SC4823S6-TR, SW13 SC4823S6-TR, SW14 SC4823S6-TR, SW2 SC4823S6-TR, SW3 SC4823S6-TR, SW4 SC4823S6-TR, SW5 SC4823S6-TR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

Commit message: :bug: improve hardware design
Parts:
- added C1: 100nF, KeysDock:C_0402, symbol components:0402,100nF
- added C2: 4.7uF, KeysDock:C_0402, symbol components:0402,4.7uF
- added C3: 10uF, KeysDock:C_0402, symbol components:0402,10uF
Connections:
- net P,+3.3: now also C1.1, C2.1, C3.1
- net P,GND: now also C1.2, C2.2, C3.2
