File: hardware/typeboard.kicad_sch (KiCad schematic)
At the start: 69 parts, among them J2 AXK6F20347YG

Commit message: :arrow_up: update to KiCAD 10.0
Parts:
- PC1: value ~ -> (none)

Commit message: :bug: improve hardware design
Parts:
- added C13, C14: 22uF, KeysDock:C_0402, symbol components:0402,22uF
Connections:
- net P,+3.3: now also C13.1, C14.1
- net P,GND: now also C13.2, C14.2
