File: hardware/keysdock.kicad_pcb (KiCad board)
At the start: 2 copper layers, 347.8 x 117.3 mm, 0 parts

Commit message: :construction: new board
Parts:
- added C1: 10uF, KeysDock:C_0402, B.Cu at (-44.0, 131.6)
- added C10: 10uF, KeysDock:C_0402, B.Cu at (-46.9, 133.4)
- added C11: 1uF, KeysDock:C_0402, B.Cu at (-46.9, 135.2)
- added C12: 4.7uF, KeysDock:C_0402, B.Cu at (-46.9, 137.1)
- added C13: 100nF, KeysDock:C_0402, B.Cu at (-46.9, 138.9)
- added C14: 1uF, KeysDock:C_0402, B.Cu at (-46.9, 140.8)
- added C15: 1uF, KeysDock:C_0402, B.Cu at (-46.9, 142.7)
- added C16: 1uF, KeysDock:C_0402, B.Cu at (-46.9, 144.5)
- added C17: 100nF, KeysDock:C_0402, B.Cu at (-91.7, 134.3)
- added C18: 4.7uF, KeysDock:C_0402, B.Cu at (-91.7, 136.2)
- added C19: 10uF, KeysDock:C_0402, B.Cu at (-91.7, 138.0)
- added C2: 3.3nF, KeysDock:C_0402, B.Cu at (-44.0, 133.4)
- added C20: 100nF, KeysDock:C_0402, B.Cu at (-91.7, 59.2)
- added C21: 4.7uF, KeysDock:C_0402, B.Cu at (-91.7, 61.1)
- added C22: 10uF, KeysDock:C_0402, B.Cu at (-91.7, 63.0)
- added C23: 100nF, KeysDock:C_0402, B.Cu at (-158.1, 59.2)
- added C24: 4.7uF, KeysDock:C_0402, B.Cu at (-158.1, 61.1)
- added C25: 10uF, KeysDock:C_0402, B.Cu at (-158.1, 63.0)
- added C26: 100nF, KeysDock:C_0402, B.Cu at (-158.1, 134.3)
- added C27: 4.7uF, KeysDock:C_0402, B.Cu at (-158.1, 136.2)
- added C28: 10uF, KeysDock:C_0402, B.Cu at (-158.1, 138.0)
- added C29: 100nF, KeysDock:C_0402, B.Cu at (-71.6, 3.50)
- added C3: 1uF, KeysDock:C_0402, B.Cu at (-44.0, 135.2)
- added C30: 4.7uF, KeysDock:C_0402, B.Cu at (-71.6, 5.35)
- added C31: 10uF, KeysDock:C_0402, B.Cu at (-71.6, 7.20)
- added C4: 22uF, KeysDock:C_0402, B.Cu at (-44.0, 137.1)
- added C5: 100nF, KeysDock:C_0402, B.Cu at (-44.0, 138.9)
- added C6: 100nF, KeysDock:C_0402, B.Cu at (-44.0, 140.8)
- added C7: 100nF, KeysDock:C_0402, B.Cu at (-44.0, 142.7)
- added C8: 4.7uF, KeysDock:C_0402, B.Cu at (-44.0, 144.5)
- added C9: 1uF, KeysDock:C_0402, B.Cu at (-46.9, 131.6)
- added D1: TPD1E10B06DPYR, KeysDock:DIO_TPD1E05U06DPYR, B.Cu at (-31.4, 169.1)
- added D2: SM4007PL, KeysDock:D_SOD-123FL, B.Cu at (-36.7, 168.6)
- added J1: TYPE-C 16PFS 2JCB1.2-H6.5 IPX8, KeysDock:USB-C-SMD_SHOUHAN_TYPE-C-16PFS-2JCB1.2-H6.5, B.Cu at (-49.7, 148.0)
- added L1: 2.2uH, KeysDock:IND-SMD_L2.5-W2.0_MHCHL2520, B.Cu at (-31.4, 166.4)
- added LED1: XL-6028RGBW-WS2812B, KeysDock:XL-6028RGBW-WS2812B, F.Cu at (83.5, 75.6)
- added LED10: XL-6028RGBW-WS2812B, KeysDock:XL-6028RGBW-WS2812B, F.Cu at (283.6, 75.6)
- added LED11: XL-6028RGBW-WS2812B, KeysDock:XL-6028RGBW-WS2812B, F.Cu at (302.6, 75.6)
- added LED12: XL-6028RGBW-WS2812B, KeysDock:XL-6028RGBW-WS2812B, F.Cu at (321.6, 75.6)
- added LED13: XL-6028RGBW-WS2812B, KeysDock:XL-6028RGBW-WS2812B, F.Cu at (340.7, 75.6)
- added LED14: XL-6028RGBW-WS2812B, KeysDock:XL-6028RGBW-WS2812B, F.Cu at (369.3, 75.6)
- added LED15: XL-6028RGBW-WS2812B, KeysDock:XL-6028RGBW-WS2812B, F.Cu at (83.5, 99.5)
- added LED16: XL-6028RGBW-WS2812B, KeysDock:XL-6028RGBW-WS2812B, F.Cu at (102.6, 99.5)
- added LED17: XL-6028RGBW-WS2812B, KeysDock:XL-6028RGBW-WS2812B, F.Cu at (121.6, 99.5)
- added LED18: XL-6028RGBW-WS2812B, KeysDock:XL-6028RGBW-WS2812B, F.Cu at (140.7, 99.5)
- added LED19: XL-6028RGBW-WS2812B, KeysDock:XL-6028RGBW-WS2812B, F.Cu at (159.7, 99.5)
- added LED2: XL-6028RGBW-WS2812B, KeysDock:XL-6028RGBW-WS2812B, F.Cu at (112.1, 75.6)
- added LED20: XL-6028RGBW-WS2812B, KeysDock:XL-6028RGBW-WS2812B, F.Cu at (178.8, 99.5)
- added LED21: XL-6028RGBW-WS2812B, KeysDock:XL-6028RGBW-WS2812B, F.Cu at (197.8, 99.5)
- added LED22: XL-6028RGBW-WS2812B, KeysDock:XL-6028RGBW-WS2812B, F.Cu at (216.9, 99.5)
- added LED23: XL-6028RGBW-WS2812B, KeysDock:XL-6028RGBW-WS2812B, F.Cu at (235.9, 99.5)
- added LED24: XL-6028RGBW-WS2812B, KeysDock:XL-6028RGBW-WS2812B, F.Cu at (255.0, 99.5)
- added LED25: XL-6028RGBW-WS2812B, KeysDock:XL-6028RGBW-WS2812B, F.Cu at (274.0, 99.5)
- added LED26: XL-6028RGBW-WS2812B, KeysDock:XL-6028RGBW-WS2812B, F.Cu at (293.1, 99.5)
- added LED27: XL-6028RGBW-WS2812B, KeysDock:XL-6028RGBW-WS2812B, F.Cu at (312.1, 99.5)
- added LED28: XL-6028RGBW-WS2812B, KeysDock:XL-6028RGBW-WS2812B, F.Cu at (340.7, 99.5)
- added LED29: XL-6028RGBW-WS2812B, KeysDock:XL-6028RGBW-WS2812B, F.Cu at (88.3, 118.5)
- added LED3: XL-6028RGBW-WS2812B, KeysDock:XL-6028RGBW-WS2812B, F.Cu at (131.2, 75.6)
- added LED30: XL-6028RGBW-WS2812B, KeysDock:XL-6028RGBW-WS2812B, F.Cu at (112.1, 118.5)
- added LED31: XL-6028RGBW-WS2812B, KeysDock:XL-6028RGBW-WS2812B, F.Cu at (131.2, 118.5)
- added LED32: XL-6028RGBW-WS2812B, KeysDock:XL-6028RGBW-WS2812B, F.Cu at (150.2, 118.5)
- added LED33: XL-6028RGBW-WS2812B, KeysDock:XL-6028RGBW-WS2812B, F.Cu at (169.2, 118.5)
- added LED34: XL-6028RGBW-WS2812B, KeysDock:XL-6028RGBW-WS2812B, F.Cu at (188.3, 118.5)
- added LED35: XL-6028RGBW-WS2812B, KeysDock:XL-6028RGBW-WS2812B, F.Cu at (207.3, 118.5)
- added LED36: XL-6028RGBW-WS2812B, KeysDock:XL-6028RGBW-WS2812B, F.Cu at (226.4, 118.5)
- added LED37: XL-6028RGBW-WS2812B, KeysDock:XL-6028RGBW-WS2812B, F.Cu at (245.4, 118.5)
- added LED38: XL-6028RGBW-WS2812B, KeysDock:XL-6028RGBW-WS2812B, F.Cu at (264.5, 118.5)
- added LED39: XL-6028RGBW-WS2812B, KeysDock:XL-6028RGBW-WS2812B, F.Cu at (283.6, 118.5)
- added LED4: XL-6028RGBW-WS2812B, KeysDock:XL-6028RGBW-WS2812B, F.Cu at (150.2, 75.6)
- added LED40: XL-6028RGBW-WS2812B, KeysDock:XL-6028RGBW-WS2812B, F.Cu at (302.6, 118.5)
- added LED41: XL-6028RGBW-WS2812B, KeysDock:XL-6028RGBW-WS2812B, F.Cu at (321.6, 118.5)
- added LED42: XL-6028RGBW-WS2812B, KeysDock:XL-6028RGBW-WS2812B, F.Cu at (345.5, 118.5)
- added LED43: XL-6028RGBW-WS2812B, KeysDock:XL-6028RGBW-WS2812B, F.Cu at (90.7, 137.6)
- added LED44: XL-6028RGBW-WS2812B, KeysDock:XL-6028RGBW-WS2812B, F.Cu at (116.9, 137.6)
- added LED45: XL-6028RGBW-WS2812B, KeysDock:XL-6028RGBW-WS2812B, F.Cu at (135.9, 137.6)
- added LED46: XL-6028RGBW-WS2812B, KeysDock:XL-6028RGBW-WS2812B, F.Cu at (155.0, 137.6)
- added LED47: XL-6028RGBW-WS2812B, KeysDock:XL-6028RGBW-WS2812B, F.Cu at (174.0, 137.6)
- added LED48: XL-6028RGBW-WS2812B, KeysDock:XL-6028RGBW-WS2812B, F.Cu at (193.1, 137.6)
- added LED49: XL-6028RGBW-WS2812B, KeysDock:XL-6028RGBW-WS2812B, F.Cu at (212.1, 137.6)
- added LED5: XL-6028RGBW-WS2812B, KeysDock:XL-6028RGBW-WS2812B, F.Cu at (169.2, 75.6)
- added LED50: XL-6028RGBW-WS2812B, KeysDock:XL-6028RGBW-WS2812B, F.Cu at (231.2, 137.6)
- added LED51: XL-6028RGBW-WS2812B, KeysDock:XL-6028RGBW-WS2812B, F.Cu at (250.2, 137.6)
- added LED52: XL-6028RGBW-WS2812B, KeysDock:XL-6028RGBW-WS2812B, F.Cu at (269.3, 137.6)
- added LED53: XL-6028RGBW-WS2812B, KeysDock:XL-6028RGBW-WS2812B, F.Cu at (288.3, 137.6)
- added LED54: XL-6028RGBW-WS2812B, KeysDock:XL-6028RGBW-WS2812B, F.Cu at (307.4, 137.6)
- added LED55: XL-6028RGBW-WS2812B, KeysDock:XL-6028RGBW-WS2812B, F.Cu at (338.3, 137.6)
- added LED56: XL-6028RGBW-WS2812B, KeysDock:XL-6028RGBW-WS2812B, F.Cu at (93.0, 156.6)
- added LED57: XL-6028RGBW-WS2812B, KeysDock:XL-6028RGBW-WS2812B, F.Cu at (121.6, 156.6)
- added LED58: XL-6028RGBW-WS2812B, KeysDock:XL-6028RGBW-WS2812B, F.Cu at (140.7, 156.6)
- added LED59: XL-6028RGBW-WS2812B, KeysDock:XL-6028RGBW-WS2812B, F.Cu at (159.7, 156.6)
- added LED6: XL-6028RGBW-WS2812B, KeysDock:XL-6028RGBW-WS2812B, F.Cu at (197.8, 75.6)
- added LED60: XL-6028RGBW-WS2812B, KeysDock:XL-6028RGBW-WS2812B, F.Cu at (178.8, 156.6)
- added LED61: XL-6028RGBW-WS2812B, KeysDock:XL-6028RGBW-WS2812B, F.Cu at (197.8, 156.6)
- added LED62: XL-6028RGBW-WS2812B, KeysDock:XL-6028RGBW-WS2812B, F.Cu at (216.9, 156.6)
- added LED63: XL-6028RGBW-WS2812B, KeysDock:XL-6028RGBW-WS2812B, F.Cu at (235.9, 156.6)
- added LED64: XL-6028RGBW-WS2812B, KeysDock:XL-6028RGBW-WS2812B, F.Cu at (255.0, 156.6)
- added LED65: XL-6028RGBW-WS2812B, KeysDock:XL-6028RGBW-WS2812B, F.Cu at (274.0, 156.6)
- added LED66: XL-6028RGBW-WS2812B, KeysDock:XL-6028RGBW-WS2812B, F.Cu at (293.1, 156.6)
- added LED67: XL-6028RGBW-WS2812B, KeysDock:XL-6028RGBW-WS2812B, F.Cu at (321.6, 156.6)
- added LED68: XL-6028RGBW-WS2812B, KeysDock:XL-6028RGBW-WS2812B, F.Cu at (350.2, 156.6)
- added LED69: XL-6028RGBW-WS2812B, KeysDock:XL-6028RGBW-WS2812B, F.Cu at (85.9, 175.7)
- added LED7: XL-6028RGBW-WS2812B, KeysDock:XL-6028RGBW-WS2812B, F.Cu at (216.9, 75.6)
- added LED70: XL-6028RGBW-WS2812B, KeysDock:XL-6028RGBW-WS2812B, F.Cu at (109.7, 175.7)
- added LED71: XL-6028RGBW-WS2812B, KeysDock:XL-6028RGBW-WS2812B, F.Cu at (133.5, 175.7)
- added LED72: XL-6028RGBW-WS2812B, KeysDock:XL-6028RGBW-WS2812B, F.Cu at (205.0, 175.7)
- added LED73: XL-6028RGBW-WS2812B, KeysDock:XL-6028RGBW-WS2812B, F.Cu at (274.0, 175.7)
- added LED74: XL-6028RGBW-WS2812B, KeysDock:XL-6028RGBW-WS2812B, F.Cu at (293.1, 175.7)
- added LED75: XL-6028RGBW-WS2812B, KeysDock:XL-6028RGBW-WS2812B, F.Cu at (312.1, 175.7)
- added LED76: XL-6028RGBW-WS2812B, KeysDock:XL-6028RGBW-WS2812B, F.Cu at (331.2, 175.7)
- added LED77: XL-6028RGBW-WS2812B, KeysDock:XL-6028RGBW-WS2812B, F.Cu at (350.2, 175.7)
- added LED78: XL-6028RGBW-WS2812B, KeysDock:XL-6028RGBW-WS2812B, F.Cu at (369.3, 175.7)
- added LED79: XL-6028RGBW-WS2812B, KeysDock:XL-6028RGBW-WS2812B, F.Cu at (54.1, 87.5)
- added LED8: XL-6028RGBW-WS2812B, KeysDock:XL-6028RGBW-WS2812B, F.Cu at (235.9, 75.6)
- added LED80: XL-6028RGBW-WS2812B, KeysDock:XL-6028RGBW-WS2812B, F.Cu at (58.1, 121.1)
- added LED81: XL-6028RGBW-WS2812B, KeysDock:XL-6028RGBW-WS2812B, F.Cu at (43.6, 87.5)
- added LED82: XL-6028RGBW-WS2812B, KeysDock:XL-6028RGBW-WS2812B, F.Cu at (372.1, 117.0)
- added LED9: XL-6028RGBW-WS2812B, KeysDock:XL-6028RGBW-WS2812B, F.Cu at (255.0, 75.6)
- added PC1: HC-1.25-4PWT, KeysDock:HC-1.25-4PWT, B.Cu at (-40.6, 177.4)
- added PC2: HC-1.25-2PWT, KeysDock:HC-1.25-2PWT, B.Cu at (-53.2, 156.7)
- added R1: 100Ω, KeysDock:R_0402, B.Cu at (-49.7, 131.6)
- added R10: 10kΩ, KeysDock:R_0402, B.Cu at (-52.6, 133.4)
- added R11: 100Ω, KeysDock:R_0402, B.Cu at (-52.6, 135.2)
- added R12: 10kΩ, KeysDock:R_0402, B.Cu at (-52.6, 137.1)
- added R13: 1.10kΩ, KeysDock:R_0402, B.Cu at (-52.6, 138.9)
- added R14: 47kΩ, KeysDock:R_0402, B.Cu at (-52.6, 140.8)
- added R15: 750Ω, KeysDock:R_0402, B.Cu at (-52.6, 142.7)
- added R16: 10kΩ, KeysDock:R_0402, B.Cu at (-52.6, 144.5)
- added R17: 3kΩ, KeysDock:R_0402, B.Cu at (-55.4, 131.6)
- added R18: 1.5kΩ, KeysDock:R_0402, B.Cu at (-55.4, 133.4)
- added R19: 1.5kΩ, KeysDock:R_0402, B.Cu at (-55.4, 135.2)
- added R2: 10kΩ, KeysDock:R_0402, B.Cu at (-49.7, 133.4)
- added R20: 100kΩ, KeysDock:R_0402, B.Cu at (-55.4, 137.1)
- added R21: 100kΩ, KeysDock:R_0402, B.Cu at (-55.4, 138.9)
- added R22: 10kΩ, KeysDock:R_0402, B.Cu at (-71.6, 9.05)
- added R23: 100Ω, KeysDock:R_0402, B.Cu at (-74.0, 77.3)
- added R3: 10kΩ, KeysDock:R_0402, B.Cu at (-49.7, 135.2)
- added R4: 22Ω, KeysDock:R_0402, B.Cu at (-49.7, 137.1)
- added R5: 100kΩ, KeysDock:R_0402, B.Cu at (-49.7, 138.9)
- added R6: 22Ω, KeysDock:R_0402, B.Cu at (-49.7, 140.8)
- added R7: 5.1kΩ, KeysDock:R_0402, B.Cu at (-49.7, 142.7)
- added R8: 5.1kΩ, KeysDock:R_0402, B.Cu at (-49.7, 144.5)
- added R9: 10kΩ, KeysDock:R_0402, B.Cu at (-52.6, 131.6)
- added S1: TS24CA, KeysDock:TS24CA, B.Cu at (-37.5, 160.6)
- added S2: TS-1088-AR02016, 160gf, KeysDock:SW_TS-1088-AR02016, B.Cu at (-37.3, 49.6)
- added S3: SSSS811101, KeysDock:SW-SMD_SSSS811101, B.Cu at (-38.4, 43.6)
- added SW1: SC4823S6-TR, KeysDock:KD-SINGLE-KEY, F.Cu at (83.5, 80.5)
- added SW10: SC4823S6-TR, KeysDock:KD-SINGLE-KEY, F.Cu at (283.6, 80.5)
- added SW11: SC4823S6-TR, KeysDock:KD-SINGLE-KEY, F.Cu at (302.6, 80.5)
- added SW12: SC4823S6-TR, KeysDock:KD-SINGLE-KEY, F.Cu at (321.6, 80.5)
- added SW13: SC4823S6-TR, KeysDock:KD-SINGLE-KEY, F.Cu at (340.7, 80.5)
- added SW14: SC4823S6-TR, KeysDock:KD-SINGLE-KEY, F.Cu at (369.3, 80.5)
- added SW15: SC4823S6-TR, KeysDock:KD-SINGLE-KEY, F.Cu at (83.5, 104.6)
- added SW16: SC4823S6-TR, KeysDock:KD-SINGLE-KEY, F.Cu at (102.6, 104.6)
- added SW17: SC4823S6-TR, KeysDock:KD-SINGLE-KEY, F.Cu at (121.6, 104.6)
- added SW18: SC4823S6-TR, KeysDock:KD-SINGLE-KEY, F.Cu at (140.7, 104.6)
- added SW19: SC4823S6-TR, KeysDock:KD-SINGLE-KEY, F.Cu at (159.7, 104.6)
- added SW2: SC4823S6-TR, KeysDock:KD-SINGLE-KEY, F.Cu at (112.1, 80.5)
- added SW20: SC4823S6-TR, KeysDock:KD-SINGLE-KEY, F.Cu at (178.8, 104.6)
- added SW21: SC4823S6-TR, KeysDock:KD-SINGLE-KEY, F.Cu at (197.8, 104.6)
- added SW22: SC4823S6-TR, KeysDock:KD-SINGLE-KEY, F.Cu at (216.9, 104.6)
- added SW23: SC4823S6-TR, KeysDock:KD-SINGLE-KEY, F.Cu at (235.9, 104.6)
- added SW24: SC4823S6-TR, KeysDock:KD-SINGLE-KEY, F.Cu at (255.0, 104.6)
- added SW25: SC4823S6-TR, KeysDock:KD-SINGLE-KEY, F.Cu at (274.0, 104.6)
- added SW26: SC4823S6-TR, KeysDock:KD-SINGLE-KEY, F.Cu at (293.1, 104.6)
- added SW27: SC4823S6-TR, KeysDock:KD-SINGLE-KEY, F.Cu at (312.1, 104.6)
- added SW28: SC4823S6-TR, KeysDock:KD-SINGLE-KEY, F.Cu at (340.7, 104.6)
- added SW29: SC4823S6-TR, KeysDock:KD-SINGLE-KEY, F.Cu at (88.3, 123.6)
- added SW3: SC4823S6-TR, KeysDock:KD-SINGLE-KEY, F.Cu at (131.2, 80.5)
- added SW30: SC4823S6-TR, KeysDock:KD-SINGLE-KEY, F.Cu at (112.1, 123.6)
- added SW31: SC4823S6-TR, KeysDock:KD-SINGLE-KEY, F.Cu at (131.2, 123.6)
- added SW32: SC4823S6-TR, KeysDock:KD-SINGLE-KEY, F.Cu at (150.2, 123.6)
- added SW33: SC4823S6-TR, KeysDock:KD-SINGLE-KEY, F.Cu at (169.2, 123.6)
- added SW34: SC4823S6-TR, KeysDock:KD-SINGLE-KEY, F.Cu at (188.3, 123.6)
- added SW35: SC4823S6-TR, KeysDock:KD-SINGLE-KEY, F.Cu at (207.3, 123.6)
- added SW36: SC4823S6-TR, KeysDock:KD-SINGLE-KEY, F.Cu at (226.4, 123.6)
- added SW37: SC4823S6-TR, KeysDock:KD-SINGLE-KEY, F.Cu at (245.4, 123.6)
- added SW38: SC4823S6-TR, KeysDock:KD-SINGLE-KEY, F.Cu at (264.5, 123.6)
- added SW39: SC4823S6-TR, KeysDock:KD-SINGLE-KEY, F.Cu at (283.6, 123.6)
- added SW4: SC4823S6-TR, KeysDock:KD-SINGLE-KEY, F.Cu at (150.2, 80.5)
- added SW40: SC4823S6-TR, KeysDock:KD-SINGLE-KEY, F.Cu at (302.6, 123.6)
- added SW41: SC4823S6-TR, KeysDock:KD-SINGLE-KEY, F.Cu at (321.6, 123.6)
- added SW42: SC4823S6-TR, KeysDock:KD-SINGLE-KEY, F.Cu at (345.5, 123.6)
- added SW43: SC4823S6-TR, KeysDock:KD-SINGLE-KEY, F.Cu at (90.7, 142.7)
- added SW44: SC4823S6-TR, KeysDock:KD-SINGLE-KEY, F.Cu at (116.9, 142.7)
- added SW45: SC4823S6-TR, KeysDock:KD-SINGLE-KEY, F.Cu at (135.9, 142.7)
- added SW46: SC4823S6-TR, KeysDock:KD-SINGLE-KEY, F.Cu at (155.0, 142.7)
- added SW47: SC4823S6-TR, KeysDock:KD-SINGLE-KEY, F.Cu at (174.0, 142.7)
- added SW48: SC4823S6-TR, KeysDock:KD-SINGLE-KEY, F.Cu at (193.1, 142.7)
- added SW49: SC4823S6-TR, KeysDock:KD-SINGLE-KEY, F.Cu at (212.1, 142.7)
- added SW5: SC4823S6-TR, KeysDock:KD-SINGLE-KEY, F.Cu at (169.2, 80.5)
- added SW50: SC4823S6-TR, KeysDock:KD-SINGLE-KEY, F.Cu at (231.2, 142.7)
- added SW51: SC4823S6-TR, KeysDock:KD-SINGLE-KEY, F.Cu at (250.2, 142.7)
- added SW52: SC4823S6-TR, KeysDock:KD-SINGLE-KEY, F.Cu at (269.3, 142.7)
- added SW53: SC4823S6-TR, KeysDock:KD-SINGLE-KEY, F.Cu at (288.3, 142.7)
- added SW54: SC4823S6-TR, KeysDock:KD-SINGLE-KEY, F.Cu at (307.4, 142.7)
- added SW55: SC4823S6-TR, KeysDock:KD-SINGLE-KEY, F.Cu at (338.3, 142.7)
- added SW56: SC4823S6-TR, KeysDock:KD-SINGLE-KEY, F.Cu at (93.0, 161.7)
- added SW57: SC4823S6-TR, KeysDock:KD-SINGLE-KEY, F.Cu at (121.6, 161.7)
- added SW58: SC4823S6-TR, KeysDock:KD-SINGLE-KEY, F.Cu at (140.7, 161.7)
- added SW59: SC4823S6-TR, KeysDock:KD-SINGLE-KEY, F.Cu at (159.7, 161.7)
- added SW6: SC4823S6-TR, KeysDock:KD-SINGLE-KEY, F.Cu at (197.8, 80.5)
- added SW60: SC4823S6-TR, KeysDock:KD-SINGLE-KEY, F.Cu at (178.8, 161.7)
- added SW61: SC4823S6-TR, KeysDock:KD-SINGLE-KEY, F.Cu at (197.8, 161.7)
- added SW62: SC4823S6-TR, KeysDock:KD-SINGLE-KEY, F.Cu at (216.9, 161.7)
- added SW63: SC4823S6-TR, KeysDock:KD-SINGLE-KEY, F.Cu at (235.9, 161.7)
- added SW64: SC4823S6-TR, KeysDock:KD-SINGLE-KEY, F.Cu at (255.0, 161.7)
- added SW65: SC4823S6-TR, KeysDock:KD-SINGLE-KEY, F.Cu at (274.0, 161.7)
- added SW66: SC4823S6-TR, KeysDock:KD-SINGLE-KEY, F.Cu at (293.1, 161.7)
- added SW67: SC4823S6-TR, KeysDock:KD-SINGLE-KEY, F.Cu at (321.6, 161.7)
- added SW68: SC4823S6-TR, KeysDock:KD-SINGLE-KEY, F.Cu at (350.2, 161.7)
- added SW69: SC4823S6-TR, KeysDock:KD-SINGLE-KEY, F.Cu at (85.9, 180.8)
- added SW7: SC4823S6-TR, KeysDock:KD-SINGLE-KEY, F.Cu at (216.9, 80.5)
- added SW70: SC4823S6-TR, KeysDock:KD-SINGLE-KEY, F.Cu at (109.7, 180.8)
- added SW71: SC4823S6-TR, KeysDock:KD-SINGLE-KEY, F.Cu at (133.5, 180.8)
- added SW72: SC4823S6-TR, KeysDock:KD-SINGLE-KEY, F.Cu at (205.0, 180.8)
- added SW73: SC4823S6-TR, KeysDock:KD-SINGLE-KEY, F.Cu at (274.0, 180.8)
- added SW74: SC4823S6-TR, KeysDock:KD-SINGLE-KEY, F.Cu at (293.1, 180.8)
- added SW75: SC4823S6-TR, KeysDock:KD-SINGLE-KEY, F.Cu at (312.1, 180.8)
- added SW76: SC4823S6-TR, KeysDock:KD-SINGLE-KEY, F.Cu at (331.2, 180.8)
- added SW77: SC4823S6-TR, KeysDock:KD-SINGLE-KEY, F.Cu at (350.2, 180.8)
- added SW78: SC4823S6-TR, KeysDock:KD-SINGLE-KEY, F.Cu at (369.3, 180.8)
- added SW8: SC4823S6-TR, KeysDock:KD-SINGLE-KEY, F.Cu at (235.9, 80.5)
- added SW9: SC4823S6-TR, KeysDock:KD-SINGLE-KEY, F.Cu at (255.0, 80.5)
- added T1: XL4067TS, KeysDock:XL4067TS, B.Cu at (-85.8, 137.7)
- added T2: XL4067TS, KeysDock:XL4067TS, B.Cu at (-85.8, 62.6)
- added T3: XL4067TS, KeysDock:XL4067TS, B.Cu at (-152.2, 62.6)
- added T4: XL4067TS, KeysDock:XL4067TS, B.Cu at (-152.2, 137.7)
- added T5: XL4067TS, KeysDock:XL4067TS, B.Cu at (-74.7, -1.75)
- added U1: TPD4E05U06DQAR, KeysDock:IC_TPD4E05U06DQAR, B.Cu at (-27.8, 166.8)
- added U2: TPS62142RGTR, KeysDock:QFN50P300X300X80-17N, B.Cu at (-45.8, 157.9)
- added U3: ESP32-C6-WROOM-1-N8, KeysDock:ESP32-C6-WROOM-1, B.Cu at (49.0, 173.8)
- added U4: BQ24074RGTR, KeysDock:QFN50P300X300X80-17N, B.Cu at (-45.8, 163.1)
- added U5: TPS22910AYZVR, KeysDock:BGA4N50P2X2_88X88X50N, B.Cu at (-23.9, 166.8)
- added U6: TLA2518IRTER, KeysDock:QFN50P300X300X80-17N, B.Cu at (-45.8, 168.4)
Other:
- outline, holes or cut-outs redrawn

Commit message: :construction: some chip layout
Parts:
- moved R23 449.2 mm to (373.5, 116.0)
- moved T3 141.1 mm to (-26.4, 126.5)
- moved C23 141.1 mm to (-32.3, 123.1)
- moved C24 141.1 mm to (-32.3, 125.0)
- moved C25 141.1 mm to (-32.3, 126.8)
- moved C26 134.2 mm to (-26.4, 108.4)
- moved C27 134.2 mm to (-26.4, 110.2)
- moved C28 134.2 mm to (-26.4, 112.1)
- moved T4 134.2 mm to (-20.5, 111.8)
- moved U6 124.7 mm to (55.0, 95.0)
- moved J1 122.5 mm to (49.0, 75.5), turned to 0 degrees
- moved C29 117.3 mm to (-2.83, 98.5)
- moved C30 117.3 mm to (-2.83, 100.4)
- moved C31 117.3 mm to (-2.83, 102.2)
- moved R22 117.3 mm to (-2.83, 104.1)
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Other:
- outline, holes or cut-outs redrawn
- board text added: "- R T +"
