File: hardware/keysdock.kicad_pcb (KiCad board)
At the start: 4 copper layers, 347.8 x 117.3 mm, 235 parts, among them J1 TYPE-C 16PFS 2JCB1.2-H6.5 IPX8, SW1 SC4823S6-TR, SW10 SC4823S6-TR, SW11 SC4823S6-TR, SW12 SC4823S6-TR, SW13 SC4823S6-TR, SW14 SC4823S6-TR, SW15 SC4823S6-TR, SW16 SC4823S6-TR, SW17 SC4823S6-TR, SW18 SC4823S6-TR, SW19 SC4823S6-TR, SW2 SC4823S6-TR, SW20 SC4823S6-TR, SW21 SC4823S6-TR, SW22 SC4823S6-TR, SW23 SC4823S6-TR, SW24 SC4823S6-TR, SW25 SC4823S6-TR, SW26 SC4823S6-TR, SW27 SC4823S6-TR, SW28 SC4823S6-TR, SW29 SC4823S6-TR, SW3 SC4823S6-TR, SW30 SC4823S6-TR, SW31 SC4823S6-TR, SW32 SC4823S6-TR, SW33 SC4823S6-TR, SW34 SC4823S6-TR, SW35 SC4823S6-TR, SW36 SC4823S6-TR, SW37 SC4823S6-TR, SW38 SC4823S6-TR, SW39 SC4823S6-TR, SW4 SC4823S6-TR, SW40 SC4823S6-TR, SW41 SC4823S6-TR, SW42 SC4823S6-TR, SW43 SC4823S6-TR, SW44 SC4823S6-TR, SW45 SC4823S6-TR, SW46 SC4823S6-TR, SW47 SC4823S6-TR, SW48 SC4823S6-TR, SW49 SC4823S6-TR, SW5 SC4823S6-TR, SW50 SC4823S6-TR, SW51 SC4823S6-TR, SW52 SC4823S6-TR, SW53 SC4823S6-TR, SW54 SC4823S6-TR, SW55 SC4823S6-TR, SW56 SC4823S6-TR, SW57 SC4823S6-TR, SW58 SC4823S6-TR, SW59 SC4823S6-TR, SW6 SC4823S6-TR, SW60 SC4823S6-TR, SW61 SC4823S6-TR, SW62 SC4823S6-TR, SW63 SC4823S6-TR, SW64 SC4823S6-TR, SW65 SC4823S6-TR, SW66 SC4823S6-TR, SW67 SC4823S6-TR, SW68 SC4823S6-TR, SW69 SC4823S6-TR, SW7 SC4823S6-TR, SW70 SC4823S6-TR, SW71 SC4823S6-TR, SW72 SC4823S6-TR, SW73 SC4823S6-TR, SW74 SC4823S6-TR, SW75 SC4823S6-TR, SW76 SC4823S6-TR, SW77 SC4823S6-TR, SW78 SC4823S6-TR, SW8 SC4823S6-TR, SW9 SC4823S6-TR, T1 XL4067TS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

Commit message: :art: add plate support for leds
Parts:
- moved LED1 3.25 mm to (58.2, 111.8)
Routing:
- net /leds/TOMO0: track 6.11 -> 3.01 mm
- net Net-(LED1-DO): track 44.9 -> 43.5 mm
- net VCC: track 2487.0 -> 2486.4 mm
