File: hardware/keysgroup.kicad_sch (KiCad schematic)
At the start: 20 parts, among them SW19 SC4823S6-TR, SW20 SC4823S6-TR, SW21 SC4823S6-TR, SW22 SC4823S6-TR, SW23 SC4823S6-TR, SW24 SC4823S6-TR, SW25 SC4823S6-TR, SW26 SC4823S6-TR, SW27 SC4823S6-TR, SW28 SC4823S6-TR, SW29 SC4823S6-TR, SW30 SC4823S6-TR, SW31 SC4823S6-TR, SW32 SC4823S6-TR, SW33 SC4823S6-TR, SW34 SC4823S6-TR, T2 XL4067TS

Commit message: :construction: new board
Parts:
- renumbered C12 to C17, C13 to C18, C14 to C19, SW19 to SW1, SW28 to SW10, SW29 to SW11, SW30 to SW12, SW31 to SW13, SW32 to SW14, SW33 to SW15, SW34 to SW16, SW20 to SW2, SW21 to SW3, SW22 to SW4, SW23 to SW5, SW24 to SW6, SW25 to SW7, SW26 to SW8, SW27 to SW9, T2 to T1

Commit message: :construction: some chip layout
Parts:
- C17: symbol components:0402,100nF -> KeysDock:0402,100nF
- C18: symbol components:0402,4.7uF -> KeysDock:0402,4.7uF
- C19: symbol components:0402,10uF -> KeysDock:0402,10uF
- T1: symbol components:XL4067TS -> KeysDock:XL4067TS
Changed lines of the file:
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@@
 	)
 	(symbol
-		(lib_id "components:0402,4.7uF")
+		(lib_id "KeysDock:0402,4.7uF")
 		(at 242.57 129.54 0)
 		(unit 1)
@@
 	)
 	(symbol
-		(lib_id "components:XL4067TS")
+		(lib_id "KeysDock:XL4067TS")
 		(at 217.17 113.03 270)
 		(unit 1)
@@
 	)
 	(symbol
-		(lib_id "components:0402,100nF")
+		(lib_id "KeysDock:0402,100nF")
 		(at 237.49 129.54 0)
 		(unit 1)
@@
 	)
 	(symbol
-		(lib_id "components:0402,10uF")
+		(lib_id "KeysDock:0402,10uF")
 		(at 247.65 129.54 0)
 		(unit 1)

Commit message: :sparkles: use net tie to construct GNDs
Parts:
- renumbered SW4 to SW10, SW6 to SW11, SW8 to SW12, SW10 to SW13, SW12 to SW14, SW14 to SW15, SW3 to SW2, SW5 to SW3, SW7 to SW4, SW9 to SW5, SW11 to SW6, SW13 to SW7, SW15 to SW8, SW2 to SW9
Connections:
- net P,+3.3 renamed +3.3V
- net P,GND renamed GNDA
