File: hardware/keysdock.kicad_sch (KiCad schematic)
At the start: 59 parts, among them J1 TYPE-C 16PFS 2JCB1.2-H6.5 IPX8, U1 ESP32-C6-WROOM-1-N8, U2 TLA2518IRTER, U3 TPS62142RGTR, U4 BQ24074RGTR, U5 TPD4E05U06DQAR, U6 TPS22910AYZVR

Commit message: :construction: receiver artifacts
Parts:
- removed C1: 1uF, KeysDock:C_0402, symbol KeysDock:0402,1uF
- removed R1, R11, R2, R3, R4: 10kΩ, KeysDock:R_0402, symbol KeysDock:0402,10kΩ
- removed R21, R22: 5.1kΩ, KeysDock:R_0402, symbol KeysDock:0402,5.1kΩ
- removed R5, R6: 100Ω, KeysDock:R_0402, symbol KeysDock:0402,100Ω
- removed S1: TS24CA, KeysDock:TS24CA, symbol KeysDock:TS24CA
- removed S2: TS-1088-AR02016, 160gf, KeysDock:SW_TS-1088-AR02016, symbol KeysDock:Tactile Button, 160gf, 12V, 50mA, 4.0mm
- removed U1: ESP32-C6-WROOM-1-N8, KeysDock:ESP32-C6-WROOM-1, symbol KeysDock:ESP32-C6-WROOM-1
- added R21, R25, R26: 4.7kΩ, KeysDock:R_0402, symbol KeysDock:0402,4.7kΩ
- added R22, R24, R27, R28, R29, R30: 200kΩ, KeysDock:R_0402, symbol KeysDock:0402,200kΩ
- added R31: 100kΩ, KeysDock:R_0402, symbol KeysDock:0402,100kΩ
- added U7: TUSB320LAIRWBR, KeysDock:TUSB320LAIRWBR, symbol KeysDock:TUSB320LAIRWBR
Connections:
- net +3.3V: now also R22.1, R24.1, R25.1, R26.1, U7.12 (VDD)
- net GND: now also R21.2, U7.10 (GND), U7.11 (~{EN}), U7.5 (ADDR); no longer U4.5 (EN2)
- net VUSB: now also R31.2
- net CHG_EN1: now reaches U4.6 (EN1)
- net USB_CC2: now reaches J1.B5 (CC2), U5.5 (D2-)
- net USB_CC2: now also U7.1 (CC1)
- net USB_CC1: now reaches J1.A5 (CC1), U5.1 (D1+)
- net USB_CC1: now also U7.2 (CC2)
- net U0RX renamed mcu/U0RX
- net U0TX renamed mcu/U0TX
- new net: R27.2, R28.1
- new net: R28.2, R29.1
- new net: R21.1, U7.3 (PORT)
- new net: R27.1, U7.4 (VBUS_DET)
- new net: R22.2, U7.9 (ID)
- new net: R30.2, R31.1
- new net: R29.2, R30.1
- new net CHG_EN2: U4.5 (EN2)
- new net USB_PWR_SCL: R25.2, U7.8 (SCL/OUT2)
- new net USB_PWR_SDA: R26.2, U7.7 (SDA/OUT1)
- new net ~{USB_PWR_INT}: R24.2, U7.6 (~{INT}/OUT3)
- no-connect marks 4 -> 2
Other:
- added sheet mcu (mcu.kicad_sch)
- moved on the sheet: R7

Commit message: :construction: finish esp32 s31 designs
Connections:
- net CHG_EN1 is gone; now on net BAT_CHG_EN1: U4.6 (EN1)
- net CHG_EN2 is gone; now on net BAT_CHG_EN2: U4.5 (EN2)
Changed lines of the file:
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@@
 		)
 	)
-	(label "CHG_EN2"
+	(label "BAT_CHG_EN2"
 		(at 245.11 191.77 180)
 		(effects
@@
 		)
 	)
-	(label "CHG_EN1"
+	(label "BAT_CHG_EN1"
 		(at 245.11 189.23 180)
 		(effects
