File: hardware/mcu.kicad_sch (KiCad schematic)
At the start: 10 parts, among them U8 ESP32-S31-WROOM-3

Commit message: :construction: finish esp32 s31 designs
Connections:
- no-connect marks 0 -> 30
Changed lines of the file:
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@@
 		(color 0 0 0 0)
+	)
+	(no_connect
+		(at 64.77 101.6)
+	)
+	(no_connect
+		(at 227.33 106.68)
+	)
+	(no_connect
+		(at 227.33 66.04)
+	)
+	(no_connect
+		(at 64.77 83.82)
+	)
+	(no_connect
+		(at 227.33 104.14)
+	)
+	(no_connect
+		(at 227.33 109.22)
+	)
+	(no_connect
+		(at 64.77 91.44)
+	)
+	(no_connect
+		(at 64.77 86.36)
+	)
+	(no_connect
+		(at 64.77 76.2)
+	)
+	(no_connect
+		(at 227.33 53.34)
+	)
+	(no_connect
+		(at 227.33 76.2)
+	)
+	(no_connect
+		(at 227.33 73.66)
+	)
+	(no_connect
+		(at 64.77 116.84)
+	)
+	(no_connect
+		(at 64.77 81.28)
+	)
+	(no_connect
+		(at 227.33 71.12)
+	)
+	(no_connect
+		(at 64.77 96.52)
+	)
+	(no_connect
+		(at 227.33 68.58)
+	)
+	(no_connect
+		(at 227.33 101.6)
+	)
+	(no_connect
+		(at 227.33 111.76)
+	)
+	(no_connect
+		(at 64.77 73.66)
+	)
+	(no_connect
+		(at 227.33 60.96)
+	)
+	(no_connect
+		(at 227.33 93.98)
+	)
+	(no_connect
+		(at 64.77 114.3)
+	)
+	(no_connect
+		(at 64.77 78.74)
+	)
+	(no_connect
+		(at 227.33 63.5)
+	)
+	(no_connect
+		(at 227.33 78.74)
+	)
+	(no_connect
+		(at 227.33 81.28)
+	)
+	(no_connect
+		(at 227.33 99.06)
+	)
+	(no_connect
+		(at 227.33 55.88)
+	)
+	(no_connect
+		(at 64.77 88.9)
 	)
 	(wire
